File: hardware/stm/stm.kicad_sch (KiCad schematic)
At the start: 23 parts, among them J1 Conn_02x07_Odd_Even, J2 OUTPUT, J3 POWER, J4 INPUT, U1 STM32L021K4Tx, U2 BU33SD5WG_TR, U3 MCP4811

Commit message: pcb done
Parts:
- added H101, H102, H103, H104: MountingHole_Pad, MountingHole:MountingHole_3.2mm_M3_Pad, symbol Mechanical:MountingHole_Pad
- C7, C8: value 0.47uF -> 1uF
Connections:
- net SYS_SWCLK is gone; now on net SWDCK: U1.24 (PA14)
- net SYS_SWDIO is gone; now on net SWDIO: U1.23 (PA13)
- net GND: now also H101.1, H102.1, H103.1, H104.1
Changed lines of the file:
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@@
 (kicad_sch (version 20230121) (generator eeschema)
   (paper "A4")
+  (junction (at 242.57 81.28) (diameter 0) (color 0 0 0 0)
+  )
   (junction (at 191.77 119.38) (diameter 0) (color 0 0 0 0)
   )
@@
   (junction (at 86.36 27.94) (diameter 0) (color 0 0 0 0)
   )
+  (junction (at 252.73 81.28) (diameter 0) (color 0 0 0 0)
+  )
   (junction (at 62.23 30.48) (diameter 0) (color 0 0 0 0)
   )
@@
   )
   (junction (at 191.77 101.6) (diameter 0) (color 0 0 0 0)
+  )
+  (junction (at 247.65 81.28) (diameter 0) (color 0 0 0 0)
   )
   (junction (at 68.58 125.73) (diameter 0) (color 0 0 0 0)
@@
     (stroke (width 0) (type default))
   )
+  (wire (pts (xy 242.57 81.28) (xy 242.57 82.55))
+    (stroke (width 0) (type default))
+  )
   (wire (pts (xy 83.82 41.91) (xy 83.82 40.64))
     (stroke (width 0) (type default))
@@
     (stroke (width 0) (type default))
   )
+  (wire (pts (xy 252.73 81.28) (xy 257.81 81.28))
+    (stroke (width 0) (type default))
+  )
   (wire (pts (xy 96.52 80.01) (xy 100.33 80.01))
     (stroke (width 0) (type default))
@@
     (stroke (width 0) (type default))
   )
+  (wire (pts (xy 257.81 81.28) (xy 257.81 80.01))
+    (stroke (width 0) (type default))
+  )
   (wire (pts (xy 208.28 101.6) (xy 195.58 101.6))
     (stroke (width 0) (type default))
   )
+  (wire (pts (xy 252.73 80.01) (xy 252.73 81.28))
+    (stroke (width 0) (type default))
+  )
   (wire (pts (xy 109.22 134.62) (xy 109.22 137.16))
     (stroke (width 0) (type default))
@@
     (stroke (width 0) (type default))
   )
+  (wire (pts (xy 247.65 80.01) (xy 247.65 81.28))
+    (stroke (width 0) (type default))
+  )
   (wire (pts (xy 207.01 21.59) (xy 198.12 21.59))
     (stroke (width 0) (type default))
@@
     (stroke (width 0) (type default))
   )
+  (wire (pts (xy 247.65 81.28) (xy 252.73 81.28))
+    (stroke (width 0) (type default))
+  )
   (wire (pts (xy 62.23 135.89) (xy 80.01 135.89))
     (stroke (width 0) (type default))
   )
+  (wire (pts (xy 242.57 81.28) (xy 247.65 81.28))
+    (stroke (width 0) (type default))
+  )
   (wire (pts (xy 110.49 27.94) (xy 97.79 27.94))
     (stroke (width 0) (type default))
@@
   )
   (wire (pts (xy 97.79 25.4) (xy 97.79 27.94))
+    (stroke (width 0) (type default))
+  )
+  (wire (pts (xy 242.57 80.01) (xy 242.57 81.28))
     (stroke (width 0) (type default))
   )
@@
     )
   )
-  (global_label "SYS_SWDIO" (shape input) (at 100.33 80.01 0) (fields_autoplaced)
+  (global_label "SWDIO" (shape input) (at 100.33 80.01 0) (fields_autoplaced)
     (effects (font (size 1.27 1.27)) (justify left))
-    (property "Intersheetrefs" "${INTERSHEET_REFS}" (at 113.6566 80.01 0)
-      (effects (font (size 1.27 1.27)) (justify left) hide)
-    )
-  )
-  (global_label "SYS_SWCLK" (shape input) (at 100.33 82.55 0) (fields_autoplaced)
+    (property "Intersheetrefs" "${INTERSHEET_REFS}" (at 109.1814 80.01 0)
+      (effects (font (size 1.27 1.27)) (justify left) hide)
+    )
+  )
+  (global_label "SWDCK" (shape input) (at 100.33 82.55 0) (fields_autoplaced)
     (effects (font (size 1.27 1.27)) (justify left))
-    (property "Intersheetrefs" "${INTERSHEET_REFS}" (at 114.0194 82.55 0)
+    (property "Intersheetrefs" "${INTERSHEET_REFS}" (at 109.7861 82.55 0)
       (effects (font (size 1.27 1.27)) (justify left) hide)
     )
@@
         (path "/99bbdb7f-82d7-4276-b8c0-426739708ec2"
           (reference "R2") (unit 1)
+        )
+      )
+    )
+  )
+  (symbol (lib_id "Mechanical:MountingHole_Pad") (at 242.57 77.47 0) (unit 1)
+    (in_bom yes) (on_board yes) (dnp no) (fields_autoplaced)
+    (property "Reference" "H101" (at 245.11 74.93 0)
+      (effects (font (size 1.27 1.27)) (justify left) hide)
+    )
+    (property "Value" "MountingHole_Pad" (at 245.11 77.47 0)
+      (effects (font (size 1.27 1.27)) (justify left) hide)
+    )
+    (property "Footprint" "MountingHole:MountingHole_3.2mm_M3_Pad" (at 242.57 77.47 0)
+      (effects (font (size 1.27 1.27)) hide)
+    )
+    (property "Datasheet" "~" (at 242.57 77.47 0)
+      (effects (font (size 1.27 1.27)) hide)
+    )
+    (pin "1")
+    (instances
+      (project "stm"
+        (path "/99bbdb7f-82d7-4276-b8c0-426739708ec2"
+          (reference "H101") (unit 1)
         )
       )
@@
     )
   )
+  (symbol (lib_id "Mechanical:MountingHole_Pad") (at 257.81 77.47 0) (unit 1)
+    (in_bom yes) (on_board yes) (dnp no) (fields_autoplaced)
+    (property "Reference" "H104" (at 260.35 74.93 0)
+      (effects (font (size 1.27 1.27)) (justify left) hide)
+    )
+    (property "Value" "MountingHole_Pad" (at 260.35 77.47 0)
+      (effects (font (size 1.27 1.27)) (justify left) hide)
+    )
+    (property "Footprint" "MountingHole:MountingHole_3.2mm_M3_Pad" (at 257.81 77.47 0)
+      (effects (font (size 1.27 1.27)) hide)
+    )
+    (property "Datasheet" "~" (at 257.81 77.47 0)
+      (effects (font (size 1.27 1.27)) hide)
+    )
+    (pin "1")
+    (instances
+      (project "stm"
+        (path "/99bbdb7f-82d7-4276-b8c0-426739708ec2"
+          (reference "H104") (unit 1)
+        )
+      )
+    )
+  )
   (symbol (lib_id "Connector_Generic:Conn_01x02") (at 213.36 36.83 0) (unit 1)
     (in_bom yes) (on_board yes) (dnp no) (fields_autoplaced)
@@
       (effects (font (size 1.27 1.27)) (justify left))
     )
-    (property "Value" "0.47uF" (at 64.77 130.8163 0)
+    (property "Value" "1uF" (at 64.77 130.8163 0)
       (effects (font (size 1.27 1.27)) (justify left))
     )
@@
         (path "/99bbdb7f-82d7-4276-b8c0-426739708ec2"
           (reference "#PWR02") (unit 1)
+        )
+      )
+    )
+  )
+  (symbol (lib_id "Mechanical:MountingHole_Pad") (at 252.73 77.47 0) (unit 1)
+    (in_bom yes) (on_board yes) (dnp no) (fields_autoplaced)
+    (property "Reference" "H103" (at 255.27 74.93 0)
+      (effects (font (size 1.27 1.27)) (justify left) hide)
+    )
+    (property "Value" "MountingHole_Pad" (at 255.27 77.47 0)
+      (effects (font (size 1.27 1.27)) (justify left) hide)
+    )
+    (property "Footprint" "MountingHole:MountingHole_3.2mm_M3_Pad" (at 252.73 77.47 0)
+      (effects (font (size 1.27 1.27)) hide)
+    )
+    (property "Datasheet" "~" (at 252.73 77.47 0)
+      (effects (font (size 1.27 1.27)) hide)
+    )
+    (pin "1")
+    (instances
+      (project "stm"
+        (path "/99bbdb7f-82d7-4276-b8c0-426739708ec2"
+          (reference "H103") (unit 1)
         )
       )
@@
     )
   )
+  (symbol (lib_id "Mechanical:MountingHole_Pad") (at 247.65 77.47 0) (unit 1)
+    (in_bom yes) (on_board yes) (dnp no) (fields_autoplaced)
+    (property "Reference" "H102" (at 250.19 74.93 0)
+      (effects (font (size 1.27 1.27)) (justify left) hide)
+    )
+    (property "Value" "MountingHole_Pad" (at 250.19 77.47 0)
+      (effects (font (size 1.27 1.27)) (justify left) hide)
+    )
+    (property "Footprint" "MountingHole:MountingHole_3.2mm_M3_Pad" (at 247.65 77.47 0)
+      (effects (font (size 1.27 1.27)) hide)
+    )
+    (property "Datasheet" "~" (at 247.65 77.47 0)
+      (effects (font (size 1.27 1.27)) hide)
+    )
+    (pin "1")
+    (instances
+      (project "stm"
+        (path "/99bbdb7f-82d7-4276-b8c0-426739708ec2"
+          (reference "H102") (unit 1)
+        )
+      )
+    )
+  )
   (symbol (lib_id "power:GND") (at 110.49 38.1 0) (mirror y) (unit 1)
     (in_bom yes) (on_board yes) (dnp no) (fields_autoplaced)
@@
         (path "/99bbdb7f-82d7-4276-b8c0-426739708ec2"
           (reference "C4") (unit 1)
+        )
+      )
+    )
+  )
+  (symbol (lib_id "power:GND") (at 242.57 82.55 0) (unit 1)
+    (in_bom yes) (on_board yes) (dnp no) (fields_autoplaced)
+    (property "Reference" "#PWR0101" (at 242.57 88.9 0)
+      (effects (font (size 1.27 1.27)) hide)
+    )
+    (property "Value" "GND" (at 242.57 87.63 0)
+      (effects (font (size 1.27 1.27)))
+    )
+    (property "Footprint" "" (at 242.57 82.55 0)
+      (effects (font (size 1.27 1.27)) hide)
+    )
+    (property "Datasheet" "" (at 242.57 82.55 0)
+      (effects (font (size 1.27 1.27)) hide)
+    )
+    (pin "1")
+    (instances
+      (project "stm"
+        (path "/99bbdb7f-82d7-4276-b8c0-426739708ec2"
+          (reference "#PWR0101") (unit 1)
         )
       )
@@
       (effects (font (size 1.27 1.27)) (justify left))
     )
-    (property "Value" "0.47uF" (at 99.06 129.5463 0)
-      (effects (font (size 1.27 1.27)) (justify left))
-    )
+    (property "Value" "1uF" (at 99.06 129.5463 0)
+      (effects (font (size 1.27 1.27)) (justify left))
+    )
